File: kicad/power_supply.kicad_sch (KiCad schematic)
At the start: 14 parts, among them U3 LMR38010

Commit message: test1: copied a capacitor into power supply
Parts:
- added C41: 100nF, LibreSolar:C_0603_1608, symbol LibreSolar:C
Connections:
- net +3V3: now also C41.1
- net GND: now also C41.2
